File: modular_segment/modular_segment.kicad_pcb (KiCad board)
At the start: 2 copper layers, 65.4 x 103.1 mm, 88 parts, among them J1 USB_B_Micro, J2 Screw_Terminal_01x02, J3 Barrel_Jack_Switch_Pin3Ring, J4 Conn_01x02_Male, J5 Conn_01x02_Male, J6 Conn_01x02_Male, J7 Conn_01x02_Male, Q1 MBT3904DW1, Q10 2N7002, Q3 2N7002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

Commit message: Preliminary design complete
Parts:
- removed AI_2, AI_3: Conn_01x03_Male, Connector_PinHeader_2.54mm:PinHeader_1x03_P2.54mm_Vertical
- added g1: LOGO, Andrew_van_dam_logo:Andrew_van_dam_logo_12mm, F.Cu at (-24.1, -11.4)
- moved AI_0 228.7 mm to (-14.7, -11.2)
- moved C8 226.2 mm to (-18.8, 7.25), turned to 270 degrees
- moved R10 225.8 mm to (-11.6, -19.1)
- moved AI_1 218.4 mm to (-10.8, -11.2)
- moved R1 210.9 mm to (-12.2, 8.20), turned to 90 degrees
- moved R2 208.5 mm to (-14.4, 8.20), turned to 90 degrees
- moved C4 183.8 mm to (13.3, 29.2), turned to 270 degrees
- moved R8 183.1 mm to (16.1, 27.1), turned to 270 degrees
- moved R5 176.5 mm to (16.6, 24.0), turned to 180 degrees
- moved R6 165.6 mm to (16.9, 30.2)
- moved R7 165.5 mm to (21.0, 27.1), turned to 90 degrees
- moved Q8 158.7 mm to (1.05, 35.8), turned to 180 degrees
- moved J_PROG1 157.3 mm to (-0.20, 17.6)
- moved R27 155.5 mm to (4.15, 35.6), turned to 90 degrees
- moved R23 152.3 mm to (6.20, 35.6), turned to 90 degrees
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Connections:
- CHAIN_OUT1 pad 1: +12V -> GND
- CHAIN_OUT1 pad 2: +3V3 -> SCL
- CHAIN_OUT1 pad 4: SCL -> +3V3
- CHAIN_OUT1 pad 5: GND -> +12V
- D1 pad 10: +12V -> Net-(D1-Pad10)
- D1 pad 6: Net-(D1-Pad6) -> +12V
- U2 pad 10: PB_2 -> ENC_0_A
- U2 pad 11: PB_3 -> ENC_0_B
- U2 pad 12: ENC_1_A -> AI_0
- U2 pad 13: ENC_1_B -> AI_1
- U2 pad 35: ENC_0_B -> Net-(U2-Pad35)
- U2 pad 36: ENC_0_A -> Net-(U2-Pad36)
- U2 pad 4: AI_0 -> ENC_1_A
- U2 pad 5: AI_1 -> ENC_1_B
- U2 pad 6: AI_2 -> PB_1
- U2 pad 7: AI_3 -> PB_3
- U2 pad 8: PB_0 -> PB_2
- U2 pad 9: PB_1 -> PB_0
Routing:
- net +3V3: track 0.00 -> 226.7 mm, vias 0 -> 6
- net GND: track 0.00 -> 170.3 mm, vias 0 -> 17
- net +12V: track 0.00 -> 162.5 mm
- net SCL: track 0.00 -> 82.8 mm, vias 0 -> 4
- net SDA: track 0.00 -> 77.5 mm, vias 0 -> 4
- net GPIO0: track 0.00 -> 76.5 mm, vias 0 -> 2
- net /Fet Driver/C1: track 0.00 -> 76.0 mm, vias 0 -> 2
- net /Fet Driver/C5: track 0.00 -> 73.2 mm, vias 0 -> 4
- net PB_0: track 0.00 -> 63.6 mm, vias 0 -> 3
- net USB_RX: track 0.00 -> 56.6 mm, vias 0 -> 4
- net PB_1: track 0.00 -> 54.4 mm, vias 0 -> 1
- net CHIP_PU: track 0.00 -> 52.6 mm, vias 0 -> 2
- net /Fet Driver/C4: track 0.00 -> 52.6 mm, vias 0 -> 2
- net /Fet Driver/C3: track 0.00 -> 52.2 mm, vias 0 -> 2
- net ENC_0_A: track 0.00 -> 51.6 mm, vias 0 -> 2
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- added copper zone on B.Cu, net GND
Other:
- board text added: "16"
- board text added: "2"
- board text added: "4"
- board text added: "8"
- board text added: "ADDR"
- board text added: "J0"
- board text added: "J1"
- board text added: "J2"
- board text added: "J3"
